File: hardware/rev-a/openpocket-rev-a.kicad_sch (KiCad schematic)
At the start: 297 parts, among them J1 ER-TFT050A3-2 FFC, J11 5.8 GHz antenna U.FL, J12 push-push microSD, J13 speaker solder pads, J14 SSD1306 128x64 OLED pads, J15 expander developer pads, J16 controls ground pads, J2 USB-C, J3 battery/NTC, J4 speaker connector, J5 master switch, J6 ELRS, J7 left gimbal, J8 right gimbal, J9 controls, Q1 dual protection FET, Q2 Q_BUZZ buzzer MOSFET, U1 ESP32-S3-MINI-1U-N8, U10 display 3V3 buck, U11 analog OSD, U12 OSD 3V3-to-5V, U13 OSD 5V-to-3V3, U14 CVBS TFT controller, U15 AMT boot flash, U16 AMT flash mux, U17 backlight boost, U18 GPIO expander 0x20, U19 GPIO expander 0x21, U2 1S charger/power path, U20 master load switch, U21 I2S speaker amplifier, U22 3V3_SD load switch, U3 1S protector, U4 fuel gauge, U5 3V3 buck-boost, U6 5V boost, U7 5V_VIDEO load switch, U8 5V_DISPLAY load switch, U9 5V_ELRS load switch, Y1 27.000MHz, Y2 27.000MHz

Commit message: feat(rev-a): add edge ground pads for controls
Parts:
- removed J16: controls ground pads, OpenPocket:EDGE-PADS-2, symbol openpocket-rev-a:J16_SOLDER-PADS-2
- added J16: left control ground pads, OpenPocket:GROUND-EDGE-11, symbol openpocket-rev-a:J16_GROUND-EDGE-11
- added J17: right control ground pads, OpenPocket:GROUND-EDGE-11, symbol openpocket-rev-a:J17_GROUND-EDGE-11
Connections:
- net GND: now also J16.1 (GND1), J16.10 (GND10), J16.11 (GND11), J16.2 (GND2), J16.3 (GND3), J16.4 (GND4), J16.5 (GND5), J16.6 (GND6), J16.7 (GND7), J16.8 (GND8), J16.9 (GND9), J17.1 (GND1), J17.10 (GND10), J17.11 (GND11), J17.2 (GND2), J17.3 (GND3), J17.4 (GND4), J17.5 (GND5), J17.6 (GND6), J17.7 (GND7), J17.8 (GND8), J17.9 (GND9)
