File: hardware/rev-a/openpocket-rev-a.kicad_sch (KiCad schematic)
At the start: 298 parts, among them J1 ER-TFT050A3-2 FFC, J11 5.8 GHz antenna U.FL, J12 push-push microSD, J13 speaker solder pads, J14 SSD1306 128x64 OLED pads, J15 expander developer pads, J16 left control ground pads, J17 right control ground pads, J2 USB-C, J3 battery/NTC, J4 speaker connector, J5 master switch, J6 ELRS, J7 left gimbal, J8 right gimbal, J9 controls, Q1 dual protection FET, Q2 Q_BUZZ buzzer MOSFET, U1 ESP32-S3-MINI-1U-N8, U10 display 3V3 buck, U11 analog OSD, U12 OSD 3V3-to-5V, U13 OSD 5V-to-3V3, U14 CVBS TFT controller, U15 AMT boot flash, U16 AMT flash mux, U17 backlight boost, U18 GPIO expander 0x20, U19 GPIO expander 0x21, U2 1S charger/power path, U20 master load switch, U21 I2S speaker amplifier, U22 3V3_SD load switch, U3 1S protector, U4 fuel gauge, U5 3V3 buck-boost, U6 5V boost, U7 5V_VIDEO load switch, U8 5V_DISPLAY load switch, U9 5V_ELRS load switch, Y1 27.000MHz, Y2 27.000MHz

Commit message: feat(rev-a): split controls into edge solder groups
Parts:
- removed J16: left control ground pads, OpenPocket:GROUND-EDGE-11, symbol openpocket-rev-a:J16_GROUND-EDGE-11
- removed J17: right control ground pads, OpenPocket:GROUND-EDGE-11, symbol openpocket-rev-a:J17_GROUND-EDGE-11
- removed J9: controls, OpenPocket:EDGE-PADS-22, symbol openpocket-rev-a:J9_SOLDER-PADS-22
- added J18: rotary encoder control pads, OpenPocket:ENCODER-CONTROL-PADS, symbol openpocket-rev-a:J18_ENCODER-CONTROL-PADS
- added J19: ARM switch pads, OpenPocket:ARM-CONTROL-PADS, symbol openpocket-rev-a:J19_ARM-CONTROL-PADS
- added J20: AUX2 three-position switch pads, OpenPocket:AUX2-CONTROL-PADS, symbol openpocket-rev-a:J20_AUX2-CONTROL-PADS
- added J21: AUX3 three-position switch pads, OpenPocket:AUX3-CONTROL-PADS, symbol openpocket-rev-a:J21_AUX3-CONTROL-PADS
- added J22: AUX4 three-position switch pads, OpenPocket:AUX4-CONTROL-PADS, symbol openpocket-rev-a:J22_AUX4-CONTROL-PADS
- added J23: AIL trim pads, OpenPocket:AIL-TRIM-PADS, symbol openpocket-rev-a:J23_AIL-TRIM-PADS
- added J24: ELE trim pads, OpenPocket:ELE-TRIM-PADS, symbol openpocket-rev-a:J24_ELE-TRIM-PADS
- added J25: THR trim pads, OpenPocket:THR-TRIM-PADS, symbol openpocket-rev-a:J25_THR-TRIM-PADS
- added J26: RUD trim pads, OpenPocket:RUD-TRIM-PADS, symbol openpocket-rev-a:J26_RUD-TRIM-PADS
- added J9: menu/UI control pads, OpenPocket:MENU-CONTROL-PADS, symbol openpocket-rev-a:J9_MENU-CONTROL-PADS
Connections:
- net CTRL_0_0: now also J9.2 (MENU_UP)
- net CTRL_0_1: now also J9.4 (MENU_DOWN)
- net CTRL_0_10: now also J22.3 (LO)
- net CTRL_0_11: now also J18.4 (ENC_PRESS)
- net CTRL_0_12: now also J23.2 (MINUS)
- net CTRL_0_13: now also J23.3 (PLUS)
- net CTRL_0_14: now also J24.2 (MINUS)
- net CTRL_0_15: now also J24.3 (PLUS)
- net CTRL_0_2: now also J9.6 (MENU_ENTER)
- net CTRL_0_3: now also J9.8 (MENU_BACK)
- net CTRL_0_4: now also J19.2 (ARM)
- net CTRL_0_5: now also J20.2 (HI)
- net CTRL_0_6: now also J20.3 (LO)
- net CTRL_0_7: now also J21.2 (HI)
- net CTRL_0_8: now also J21.3 (LO)
- net CTRL_0_9: now also J22.2 (HI)
- net CTRL_1_0: now also J25.2 (MINUS)
- net CTRL_1_1: now also J25.3 (PLUS)
- net CTRL_1_2: now also J26.2 (MINUS)
- net CTRL_1_3: now also J26.3 (PLUS)
- net CTRL_1_4: now also J18.1 (ENC_A)
- net CTRL_1_5: now also J18.3 (ENC_B)
- net GND: now also J18.2 (G_ENC_A), J18.5 (G_ENC_PRESS), J19.1 (G_ARM), J20.1 (G), J21.1 (G), J22.1 (G), J23.1 (G), J24.1 (G), J25.1 (G), J26.1 (G), J9.1 (G_UP), J9.3 (G_DN), J9.5 (G_ENT), J9.7 (G_BACK)

Commit message: fix(rev-a): regenerate schematic for battery rail
Connections:
- net BAT_PROTECTED is gone; now on net BAT_RAW: C31.1, R55.1, U2.13 (BAT), U2.14 (BAT), U4.3 (VDD)
